File: CANTerm-Female-SMD/CANTerm-Female-SMD.kicad_sch (KiCad schematic)
At the start: 2 parts, among them J1 Conn_01x03_Female

Commit message: Added Gerber and images
Parts:
- R1: LCSC part number (none) -> C22787
Changed lines of the file:
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@@
+      (effects (font (size 1.27 1.27)) hide)
+    )
+    (property "LCSC part number" "C22787" (id 4) (at 102.87 81.28 90)
       (effects (font (size 1.27 1.27)) hide)
     )
