File: CANTerm-Female-THT/CANTerm-Female-THT.kicad_pcb (KiCad board)
At the start: 2 copper layers, 10.2 x 19 mm, 2 parts, among them J1 Conn_01x03_Female

Commit message: Added Gerber and images
Other:
- board text added: "CAN Terminate SMD to Female Dupont tauseefafraz.com"
Changed lines of the file:
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@@
       (outputformat 1)
       (mirror false)
-      (drillshape 1)
+      (drillshape 0)
       (scaleselection 1)
-      (outputdirectory "")
+      (outputdirectory "Gerber Files/")
     )
   )
@@
   (gr_line (start 154.94 93.58) (end 144.78 93.58) (layer "Edge.Cuts") (width 0.1))
   (gr_line (start 144.78 93.58) (end 144.78 112.63) (layer "Edge.Cuts") (width 0.1))
+  (gr_text "CAN Terminate SMD to Female Dupont\ntauseefafraz.com" (at 149.86 104.14) (layer "B.SilkS")
+    (effects (font (size 0.3 0.3) (thickness 0.075)) (justify mirror))
+  )
   (segment (start 146.035 96.52) (end 146.035 100.315) (width 0.25) (layer "F.Cu") (net 1))
   (segment (start 146.035 100.315) (end 147.32 101.6) (width 0.25) (layer "F.Cu") (net 1))
