File: CANTerm-Male-SMD/CANTerm-Male-SMD.kicad_pcb (KiCad board)
At the start: 2 copper layers, 10.2 x 17.8 mm, 2 parts, among them J1 Conn_01x03_Male

Commit message: Added Gerber and images
Other:
- board text added: "CAN Terminate SMD to Female Dupont tauseefafraz.com"
Changed lines of the file:
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@@
       (outputformat 1)
       (mirror false)
-      (drillshape 1)
+      (drillshape 0)
       (scaleselection 1)
-      (outputdirectory "")
+      (outputdirectory "Gerber Files/")
     )
   )
@@
   (gr_line (start 144.78 90.17) (end 134.62 90.17) (layer "Edge.Cuts") (width 0.1))
   (gr_line (start 144.78 107.95) (end 144.78 90.17) (layer "Edge.Cuts") (width 0.1))
+  (gr_text "CAN Terminate SMD to Female Dupont\ntauseefafraz.com" (at 139.7 99.06) (layer "B.SilkS")
+    (effects (font (size 0.3 0.3) (thickness 0.075)) (justify mirror))
+  )
   (segment (start 140.6125 92.71) (end 142.225 94.3225) (width 0.25) (layer "F.Cu") (net 1))
   (segment (start 142.225 94.3225) (end 142.225 96.52) (width 0.25) (layer "F.Cu") (net 1))
