File: CANTerm-Male-THT/CANTerm-Male-THT.kicad_pcb (KiCad board)
At the start: 2 copper layers, 10.2 x 19.5 mm, 2 parts, among them J1 Conn_01x03_Male

Commit message: Added Gerber and images
Other:
- board size 10.2 x 19.5 mm -> 10.2 x 19 mm
- board text added: "CAN Terminate SMD to Female Dupont tauseefafraz.com"
Changed lines of the file:
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@@
       (outputformat 1)
       (mirror false)
-      (drillshape 1)
+      (drillshape 0)
       (scaleselection 1)
-      (outputdirectory "")
+      (outputdirectory "Gerber Files/")
     )
   )
@@
   )
   (gr_line (start 124.46 98.56) (end 124.46 79.51) (layer "Edge.Cuts") (width 0.1))
-  (gr_line (start 134.62 99.06) (end 124.46 99.06) (layer "Edge.Cuts") (width 0.1))
+  (gr_line (start 134.62 98.56) (end 124.46 98.56) (layer "Edge.Cuts") (width 0.1))
   (gr_line (start 134.62 79.51) (end 134.62 98.56) (layer "Edge.Cuts") (width 0.1))
   (gr_line (start 124.46 79.51) (end 134.62 79.51) (layer "Edge.Cuts") (width 0.1))
+  (gr_text "CAN Terminate SMD to Female Dupont\ntauseefafraz.com" (at 129.54 90.17) (layer "B.SilkS")
+    (effects (font (size 0.3 0.3) (thickness 0.075)) (justify mirror))
+  )
   (segment (start 133.35 86.345) (end 132.065 87.63) (width 0.25) (layer "F.Cu") (net 1))
   (segment (start 133.35 82.55) (end 133.35 86.345) (width 0.25) (layer "F.Cu") (net 1))
